File: AHT20.brd (EAGLE design)
At the start: 25.4 x 17.8 mm, 19 parts, among them U1 AHT20

Commit message: Starting to handle text alignment, monospace font
Other:
- board text added: "Hello"
Changed lines of the file:
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@@
 <wire x1="22.86" y1="17.78" x2="2.54" y2="17.78" width="0" layer="20"/>
 <wire x1="2.54" y1="17.78" x2="0" y2="15.24" width="0" layer="20" curve="90"/>
-<text x="8.89" y="0.889" size="1.016" layer="21" font="vector" ratio="14" align="center">VIN</text>
+<text x="8.89" y="0.889" size="1.016" layer="172" font="fixed" ratio="14" align="center">VIN</text>
 <text x="11.43" y="4.191" size="1.016" layer="172" font="vector" ratio="14" align="center">GND</text>
-<text x="14.097" y="0.889" size="1.016" layer="21" font="vector" ratio="14" align="center">SCL</text>
-<text x="16.637" y="4.191" size="1.016" layer="21" font="vector" ratio="14" align="center">SDA</text>
+<text x="14.097" y="0.889" size="1.016" layer="172" font="fixed" ratio="14" align="center">SCL</text>
+<text x="16.637" y="4.191" size="1.016" layer="172" font="fixed" ratio="14" align="center">SDA</text>
 <text x="12.7" y="16.51" size="1.778" layer="172" ratio="15" rot="R12" align="center">AHT20</text>
 <text x="14.351" y="14.605" size="1.143" layer="172" ratio="15" align="center">Temp &amp; Humidity</text>
@@
 addr
 0x38</text>
+<text x="7.747" y="11.303" size="0.508" layer="172" ratio="15" rot="R15" align="center">Hello</text>
+<text x="7.747" y="11.811" size="0.508" layer="172" ratio="15" rot="R353" align="bottom-center">Hello</text>
+<text x="7.747" y="10.795" size="0.508" layer="172" ratio="15" rot="R352" align="top-center">Hello</text>
+<text x="6.731" y="11.303" size="0.508" layer="172" ratio="15" rot="R355" align="center-right">Hello</text>
+<text x="6.731" y="11.811" size="0.508" layer="172" ratio="15" rot="R3" align="bottom-right">Hello</text>
+<text x="6.731" y="10.795" size="0.508" layer="172" ratio="15" rot="R31" align="top-right">Hello</text>
+<text x="8.763" y="11.303" size="0.508" layer="172" ratio="15" rot="R357" align="center-left">Hello</text>
+<text x="8.763" y="11.811" size="0.508" layer="172" ratio="15" rot="R22">Hello</text>
+<text x="8.763" y="10.795" size="0.508" layer="172" ratio="15" rot="R338" align="top-left">Hello</text>
 </plain>
 <attributes>
